File: T1_proyecto/ppg.brd (EAGLE design)
At the start: 50 x 50 mm, 9 parts

Commit message: remove extra LED/R
Parts:
- removed LED5MM2: (no value), led:LED5MM
- removed RH2: (no value), rcl:VMTA55
- moved LED5MM1 10.0 mm to (25.0, 18.0), turned to 180 degrees
Connections:
- removed net N$1: LED5MM2.A, RH2.2
- net GND: no longer LED5MM2.K
- net N$5: no longer RH2.1
Changed lines of the file:
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@@
 <attribute name="VALUE" x="43.825" y="12.46" size="1.27" layer="28" rot="MR90"/>
 </element>
-<element name="LED5MM1" library="led" library_urn="urn:adsk.eagle:library:259" package="LED5MM" package3d_urn="urn:adsk.eagle:package:15799/2" value=" " x="33" y="24" smashed="yes">
-<attribute name="NAME" x="36.175" y="24.5334" size="1.27" layer="25" ratio="10"/>
-<attribute name="POPULARITY" value="93" x="54.59" y="20.19" size="1.778" layer="27" display="off"/>
-<attribute name="VALUE" x="36.2004" y="22.1966" size="1.27" layer="27" ratio="10"/>
+<element name="LED5MM1" library="led" library_urn="urn:adsk.eagle:library:259" package="LED5MM" package3d_urn="urn:adsk.eagle:package:15799/2" value=" " x="25" y="18" smashed="yes" rot="R180">
+<attribute name="NAME" x="21.825" y="17.4666" size="1.27" layer="25" ratio="10" rot="R180"/>
+<attribute name="POPULARITY" value="93" x="3.41" y="21.81" size="1.778" layer="27" rot="R180" display="off"/>
+<attribute name="VALUE" x="21.7996" y="19.8034" size="1.27" layer="27" ratio="10" rot="R180"/>
 </element>
 <element name="RH1" library="rcl" library_urn="urn:adsk.eagle:library:334" package="VMTA55" package3d_urn="urn:adsk.eagle:package:26121/2" value="" x="16" y="12.5" smashed="yes" rot="R180">
@@
 <attribute name="VALUE" x="23.095" y="0.206" size="1.27" layer="27" ratio="10"/>
 </element>
-<element name="LED5MM2" library="led" library_urn="urn:adsk.eagle:library:259" package="LED5MM" package3d_urn="urn:adsk.eagle:package:15799/2" value=" " x="15" y="18" smashed="yes" rot="R180">
-<attribute name="NAME" x="11.825" y="17.4666" size="1.27" layer="25" ratio="10" rot="R180"/>
-<attribute name="POPULARITY" value="93" x="15" y="18" size="1.778" layer="27" rot="R180" display="off"/>
-<attribute name="VALUE" x="11.7996" y="19.8034" size="1.27" layer="27" ratio="10" rot="R180"/>
-</element>
-<element name="RH2" library="rcl" library_urn="urn:adsk.eagle:library:334" package="VMTA55" package3d_urn="urn:adsk.eagle:package:26121/2" value="" x="16" y="18" smashed="yes" rot="R180">
-<attribute name="NAME" x="19.175" y="16.095" size="1.27" layer="25" ratio="10" rot="R180"/>
-<attribute name="POPULARITY" value="0" x="16" y="18" size="1.778" layer="27" rot="R180" display="off"/>
-<attribute name="SPICEPREFIX" value="R" x="16" y="18" size="1.778" layer="27" rot="R180" display="off"/>
-<attribute name="VALUE" x="19.175" y="18.635" size="1.27" layer="27" ratio="10" rot="R180"/>
-</element>
 </elements>
 <signals>
@@
 <contactref element="D1" pad="A"/>
 <contactref element="LED3MM2" pad="K"/>
-<contactref element="LED5MM2" pad="K"/>
 <wire x1="47" y1="13.73" x2="47" y2="16.27" width="0" layer="19" extent="1-1"/>
-<wire x1="34.27" y1="24" x2="47" y2="16.27" width="0" layer="19" extent="1-1"/>
-<wire x1="31.27" y1="13" x2="34.27" y2="24" width="0" layer="19" extent="1-1"/>
+<wire x1="23.73" y1="18" x2="47" y2="16.27" width="0" layer="19" extent="1-1"/>
+<wire x1="31.27" y1="13" x2="23.73" y2="18" width="0" layer="19" extent="1-1"/>
 <wire x1="30.08" y1="3" x2="31.27" y2="13" width="0" layer="19" extent="1-1"/>
-<wire x1="13.73" y1="18" x2="31.27" y2="13" width="0" layer="19" extent="1-1"/>
 </signal>
 <signal name="N$4">
@@
 <contactref element="RH1" pad="2"/>
 <contactref element="LED5MM1" pad="A"/>
-<wire x1="10.92" y1="12.5" x2="31.73" y2="24" width="0" layer="19" extent="1-1"/>
+<wire x1="10.92" y1="12.5" x2="26.27" y2="18" width="0" layer="19" extent="1-1"/>
 </signal>
 <signal name="N$5">
@@
 <contactref element="D1" pad="C"/>
 <contactref element="RH1" pad="1"/>
-<contactref element="RH2" pad="1"/>
-<wire x1="21.08" y1="12.5" x2="21.08" y2="18" width="0" layer="19" extent="1-1"/>
-<wire x1="5.5" y1="14.73" x2="21.08" y2="12.5" width="0" layer="19" extent="1-1"/>
+<wire x1="19.92" y1="3" x2="21.08" y2="12.5" width="0" layer="19" extent="1-1"/>
+<wire x1="8.92" y1="7.3" x2="19.92" y2="3" width="0" layer="19" extent="1-1"/>
+<wire x1="5.5" y1="14.73" x2="8.92" y2="7.3" width="0" layer="19" extent="1-1"/>
 <wire x1="5.5" y1="17.27" x2="5.5" y2="14.73" width="0" layer="19" extent="1-1"/>
-<wire x1="8.92" y1="7.3" x2="21.08" y2="12.5" width="0" layer="19" extent="1-1"/>
-<wire x1="19.92" y1="3" x2="8.92" y2="7.3" width="0" layer="19" extent="1-1"/>
-</signal>
-<signal name="N$1">
-<contactref element="LED5MM2" pad="A"/>
-<contactref element="RH2" pad="2"/>
-<wire x1="10.92" y1="18" x2="16.27" y2="18" width="0" layer="19" extent="1-1"/>
 </signal>
 </signals>

Commit message: update T1
Parts:
- moved GND 15.2 mm to (33.0, 9.00)
- moved LED3MM2 14.0 mm to (16.0, 12.0)
- moved LED5MM1 12.5 mm to (14.0, 24.0)
- moved D1 9.06 mm to (16.0, 2.00)
- moved VI 8.54 mm to (2.50, 8.00)
- moved RH1 6.32 mm to (14.0, 18.5)
- moved RV1 2.24 mm to (10.5, 9.30)
Other:
- board size 50 x 50 mm -> 36 x 36 mm
